Commit message: updated

File: task6/ex01/ros2_ws/src/robot_description/urdf/gazebo.urdf.xacro (robot description, xacro)
@@ -17,4 +17,16 @@
       <odom_publish_frequency>50</odom_publish_frequency>
     </plugin> -->
+    <!-- <plugin
+      filename="gz-sim-pose-publisher-system"
+      name="gz::sim::systems::PosePublisher">
+      <publish_link_pose>true</publish_link_pose>
+      <publish_sensor_pose>true</publish_sensor_pose>
+      <publish_collision_pose>false</publish_collision_pose>
+      <publish_visual_pose>false</publish_visual_pose>
+      <publish_nested_model_pose>false</publish_nested_model_pose>
+      <use_pose_vector_msg>true</use_pose_vector_msg>
+      <static_publisher>true</static_publisher>
+      <static_update_frequency>1</static_update_frequency>
+    </plugin> -->
     <plugin
       filename="gz-sim-joint-state-publisher-system"
@@ -34,11 +46,5 @@
       filename="gz-sim-sensors-system"
       name="gz::sim::systems::Sensors">
-      <!-- <render_engine>ogre2</render_engine> -->
-      <ros>
-        <namespace>/</namespace>
-      </ros>
-      <topic_name>scan</topic_name>
-      <frame_name>laser_frame</frame_name>  <!-- Фрейм для сообщений -->
-      <radiation_type>infrared</radiation_type>
+      <render_engine>ogre2</render_engine>
     </plugin>
   </gazebo>

File: task6/ex01/ros2_ws/src/robot_description/urdf/robot.urdf.xacro (robot description, xacro)
@@ -90,4 +90,185 @@
     <material>Gazebo/Orange</material>
   </gazebo>
+  <joint name="left_wheel_joint" type="continuous">
+    <parent link="base_link" />
+    <child link="left_wheel" />
+    <origin xyz="0 ${wheel_offset_y} 0" rpy="-${pi/2} 0 0" />
+    <axis xyz="0 0 1" />
+  </joint>
+  <link name="left_wheel">
+    <visual>
+      <geometry>
+        <cylinder radius="${wheel_radius}" length="${wheel_thickness}" />
+      </geometry>
+      <material name="blue" />
+    </visual>
+    <collision>
+      <geometry>
+        <sphere radius="${wheel_radius}" />
+      </geometry>
+    </collision>
+    <inertial>
+      <origin xyz="0 0 0" rpy="0 0 0" />
+      <mass value="${wheel_mass}" />
+      <inertia
+        ixx="${(1/12) * wheel_mass * (3*wheel_radius*wheel_radius + wheel_thickness*wheel_thickness)}"
+        ixy="0.0" ixz="0.0"
+        iyy="${(1/12) * wheel_mass * (3*wheel_radius*wheel_radius + wheel_thickness*wheel_thickness)}"
+        iyz="0.0"
+        izz="${(1/2) * wheel_mass * (wheel_radius*wheel_radius)}" />
+    </inertial>
+  </link>
+  <gazebo reference="left_wheel">
+    <material>Gazebo/Blue</material>
+  </gazebo>
+  <joint name="right_wheel_joint" type="continuous">
+    <parent link="base_link" />
+    <child link="right_wheel" />
+    <origin xyz="0 ${-wheel_offset_y} 0" rpy="${pi/2} 0 0" />
+    <axis xyz="0 0 -1" />
+  </joint>
+  <link name="right_wheel">
+    <visual>
+      <geometry>
+        <cylinder radius="${wheel_radius}" length="${wheel_thickness}" />
+      </geometry>
+      <material name="blue" />
+    </visual>
+    <collision>
+      <geometry>
+        <sphere radius="${wheel_radius}" />
+      </geometry>
+    </collision>
+    <inertial>
+      <origin xyz="0 0 0" rpy="0 0 0" />
+      <mass value="${wheel_mass}" />
+      <inertia
+        ixx="${(1/12) * wheel_mass * (3*wheel_radius*wheel_radius + wheel_thickness*wheel_thickness)}"
+        ixy="0.0" ixz="0.0"
+        iyy="${(1/12) * wheel_mass * (3*wheel_radius*wheel_radius + wheel_thickness*wheel_thickness)}"
+        iyz="0.0"
+        izz="${(1/2) * wheel_mass * (wheel_radius*wheel_radius)}" />
+    </inertial>
+  </link>
+  <gazebo reference="right_wheel">
+    <material>Gazebo/Blue</material>
+  </gazebo>
+  <joint name="caster_wheel_joint" type="fixed">
+    <parent link="chassis" />
+    <child link="caster_wheel" />
+    <origin xyz="${caster_wheel_offset_x} 0 ${caster_wheel_offset_z}" />
+  </joint>
+  <link name="caster_wheel">
+    <visual>
+      <geometry>
+        <sphere radius="${caster_wheel_radius}" />
+      </geometry>
+      <material name="white" />
+    </visual>
+    <collision>
+      <geometry>
+        <sphere radius="${caster_wheel_radius}" />
+      </geometry>
+    </collision>
+    <inertial>
+      <origin xyz="0 0 0" rpy="0 0 0" />
+      <mass value="${caster_wheel_mass}" />
+      <inertia ixx="${(2/5) * caster_wheel_mass * (caster_wheel_radius*caster_wheel_radius)}"
+        ixy="0.0" ixz="0.0"
+        iyy="${(2/5) * caster_wheel_mass * (caster_wheel_radius*caster_wheel_radius)}" iyz="0.0"
+        izz="${(2/5) * caster_wheel_mass * (caster_wheel_radius*caster_wheel_radius)}" />
+    </inertial>
+  </link>
+  <gazebo reference="caster_wheel">
+    <material>Gazebo/White</material>
+    <mu1 value="0.001" />
+    <mu2 value="0.001" />
+  </gazebo>
+  <!-- Первая антенна (правая) -->
+  <link name="antenna_1">
+    <inertial>
+      <origin xyz="0 0 ${antenna_length/2}" rpy="0 0 0" />
+      <mass value="${antenna_mass}" />
+      <inertia
+        ixx="${(1/12) * antenna_mass * (3*antenna_radius*antenna_radius + antenna_length*antenna_length)}"
+        ixy="0.0" ixz="0.0"
+        iyy="${(1/12) * antenna_mass * (3*antenna_radius*antenna_radius + antenna_length*antenna_length)}"
+        iyz="0.0"
+        izz="${(1/2) * antenna_mass * antenna_radius*antenna_radius}" />
+    </inertial>
+    <visual>
+      <origin xyz="0 0 ${antenna_length/2}" rpy="0 0 0" />
+      <geometry>
+        <cylinder radius="${antenna_radius}" length="${antenna_length}" />
+      </geometry>
+      <material name="${antenna_color}" />
+    </visual>
+    <collision>
+      <origin xyz="0 0 ${antenna_length/2}" rpy="0 0 0" />
+      <geometry>
+        <cylinder radius="${antenna_radius}" length="${antenna_length}" />
+      </geometry>
+    </collision>
+  </link>
+  <joint name="antenna_1_joint" type="fixed">
+    <parent link="chassis" />
+    <child link="antenna_1" />
+    <origin xyz="${antenna1_x} ${antenna1_y} ${antenna1_z}" rpy="0 0 0" />
+  </joint>
+  <!-- Вторая антенна (левая) -->
+  <link name="antenna_2">
+    <inertial>
+      <origin xyz="0 0 ${antenna_length/2}" rpy="0 0 0" />
+      <mass value="${antenna_mass}" />
+      <inertia
+        ixx="${(1/12) * antenna_mass * (3*antenna_radius*antenna_radius + antenna_length*antenna_length)}"
+        ixy="0.0" ixz="0.0"
+        iyy="${(1/12) * antenna_mass * (3*antenna_radius*antenna_radius + antenna_length*antenna_length)}"
+        iyz="0.0"
+        izz="${(1/2) * antenna_mass * antenna_radius*antenna_radius}" />
+    </inertial>
+    <visual>
+      <origin xyz="0 0 ${antenna_length/2}" rpy="0 0 0" />
+      <geometry>
+        <cylinder radius="${antenna_radius}" length="${antenna_length}" />
+      </geometry>
+      <material name="${antenna_color}" />
+    </visual>
+    <collision>
+      <origin xyz="0 0 ${antenna_length/2}" rpy="0 0 0" />
+      <geometry>
+        <cylinder radius="${antenna_radius}" length="${antenna_length}" />
+      </geometry>
+    </collision>
+  </link>
+  <joint name="antenna_2_joint" type="fixed">
+    <parent link="chassis" />
+    <child link="antenna_2" />
+    <origin xyz="${antenna2_x} ${antenna2_y} ${antenna2_z}" rpy="0 0 0" />
+  </joint>
+  <!-- Gazebo материалы для антенн -->
+  <gazebo reference="antenna_1">
+    <material>Gazebo/Black</material>
+  </gazebo>
+  <gazebo reference="antenna_2">
+    <material>Gazebo/Black</material>
+  </gazebo>
+  <link name="laser_frame">
+    <visual>
+      <geometry>
+        <cylinder radius="${laser_radius}" length="${laser_length}" />
+      </geometry>
+      <material name="black" />
+    </visual>
+    <collision>
+      <geometry>
+        <cylinder radius="${laser_radius}" length="${laser_length}" />
+      </geometry>
+    </collision>
+    <inertial>
+      <mass value="0.1" />
+      <inertia ixx="1e-3" ixy="0" ixz="0" iyy="1e-3" iyz="0" izz="1e-3" />
+    </inertial>
+  </link>
   <joint name="laser_joint" type="fixed">
     <parent link="chassis" />
@@ -95,26 +276,10 @@
     <origin xyz="${chassis_length} 0 ${chassis_height/2}" rpy="0 0 0" />
   </joint>
-  <link name="laser_frame">
-    <visual>
-      <geometry>
-        <cylinder radius="${laser_radius}" length="${laser_length}" />
-      </geometry>
-      <material name="black" />
-    </visual>
-    <collision>
-      <geometry>
-        <cylinder radius="${laser_radius}" length="${laser_length}" />
-      </geometry>
-    </collision>
-    <inertial>
-      <mass value="0.1" />
-      <inertia ixx="1e-3" ixy="0" ixz="0" iyy="1e-3" iyz="0" izz="1e-3" />
-    </inertial>
-  </link>
   <gazebo reference="laser_frame">
-    <sensor name='gpu_lidar' type='gpu_lidar'>
-      <pose relative_to='laser_frame'>0 0 0 0 0 0</pose>
+    <sensor name='laser_frame' type='gpu_lidar'>
       <topic>
         scan</topic>
+      <!-- <gz_frame_id>laser_frame</gz_frame_id> -->
+      <pose relative_to='laser_frame'>0 0 0 0 0 0</pose>
       <update_rate>
         5</update_rate>
@@ -143,169 +308,6 @@
       <visualize>
         true</visualize>
+      <!-- <frame name="laser_frame">laser_frame</frame> -->
     </sensor>
   </gazebo>
-  <joint name="left_wheel_joint" type="continuous">
-    <parent link="base_link" />
-    <child link="left_wheel" />
-    <origin xyz="0 ${wheel_offset_y} 0" rpy="-${pi/2} 0 0" />
-    <axis xyz="0 0 1" />
-  </joint>
-  <link name="left_wheel">
-    <visual>
-      <geometry>
-        <cylinder radius="${wheel_radius}" length="${wheel_thickness}" />
-      </geometry>
-      <material name="blue" />
-    </visual>
-    <collision>
-      <geometry>
-        <sphere radius="${wheel_radius}" />
-      </geometry>
-    </collision>
-    <inertial>
-      <origin xyz="0 0 0" rpy="0 0 0" />
-      <mass value="${wheel_mass}" />
-      <inertia
-        ixx="${(1/12) * wheel_mass * (3*wheel_radius*wheel_radius + wheel_thickness*wheel_thickness)}"
-        ixy="0.0" ixz="0.0"
-        iyy="${(1/12) * wheel_mass * (3*wheel_radius*wheel_radius + wheel_thickness*wheel_thickness)}"
-        iyz="0.0"
-        izz="${(1/2) * wheel_mass * (wheel_radius*wheel_radius)}" />
-    </inertial>
-  </link>
-  <gazebo reference="left_wheel">
-    <material>Gazebo/Blue</material>
-  </gazebo>
-  <joint name="right_wheel_joint" type="continuous">
-    <parent link="base_link" />
-    <child link="right_wheel" />
-    <origin xyz="0 ${-wheel_offset_y} 0" rpy="${pi/2} 0 0" />
-    <axis xyz="0 0 -1" />
-  </joint>
-  <link name="right_wheel">
-    <visual>
-      <geometry>
-        <cylinder radius="${wheel_radius}" length="${wheel_thickness}" />
-      </geometry>
-      <material name="blue" />
-    </visual>
-    <collision>
-      <geometry>
-        <sphere radius="${wheel_radius}" />
-      </geometry>
-    </collision>
-    <inertial>
-      <origin xyz="0 0 0" rpy="0 0 0" />
-      <mass value="${wheel_mass}" />
-      <inertia
-        ixx="${(1/12) * wheel_mass * (3*wheel_radius*wheel_radius + wheel_thickness*wheel_thickness)}"
-        ixy="0.0" ixz="0.0"
-        iyy="${(1/12) * wheel_mass * (3*wheel_radius*wheel_radius + wheel_thickness*wheel_thickness)}"
-        iyz="0.0"
-        izz="${(1/2) * wheel_mass * (wheel_radius*wheel_radius)}" />
-    </inertial>
-  </link>
-  <gazebo reference="right_wheel">
-    <material>Gazebo/Blue</material>
-  </gazebo>
-  <joint name="caster_wheel_joint" type="fixed">
-    <parent link="chassis" />
-    <child link="caster_wheel" />
-    <origin xyz="${caster_wheel_offset_x} 0 ${caster_wheel_offset_z}" />
-  </joint>
-  <link name="caster_wheel">
-    <visual>
-      <geometry>
-        <sphere radius="${caster_wheel_radius}" />
-      </geometry>
-      <material name="white" />
-    </visual>
-    <collision>
-      <geometry>
-        <sphere radius="${caster_wheel_radius}" />
-      </geometry>
-    </collision>
-    <inertial>
-      <origin xyz="0 0 0" rpy="0 0 0" />
-      <mass value="${caster_wheel_mass}" />
-      <inertia ixx="${(2/5) * caster_wheel_mass * (caster_wheel_radius*caster_wheel_radius)}"
-        ixy="0.0" ixz="0.0"
-        iyy="${(2/5) * caster_wheel_mass * (caster_wheel_radius*caster_wheel_radius)}" iyz="0.0"
-        izz="${(2/5) * caster_wheel_mass * (caster_wheel_radius*caster_wheel_radius)}" />
-    </inertial>
-  </link>
-  <gazebo reference="caster_wheel">
-    <material>Gazebo/White</material>
-    <mu1 value="0.001" />
-    <mu2 value="0.001" />
-  </gazebo>
-  <!-- Первая антенна (правая) -->
-  <link name="antenna_1">
-    <inertial>
-      <origin xyz="0 0 ${antenna_length/2}" rpy="0 0 0" />
-      <mass value="${antenna_mass}" />
-      <inertia
-        ixx="${(1/12) * antenna_mass * (3*antenna_radius*antenna_radius + antenna_length*antenna_length)}"
-        ixy="0.0" ixz="0.0"
-        iyy="${(1/12) * antenna_mass * (3*antenna_radius*antenna_radius + antenna_length*antenna_length)}"
-        iyz="0.0"
-        izz="${(1/2) * antenna_mass * antenna_radius*antenna_radius}" />
-    </inertial>
-    <visual>
-      <origin xyz="0 0 ${antenna_length/2}" rpy="0 0 0" />
-      <geometry>
-        <cylinder radius="${antenna_radius}" length="${antenna_length}" />
-      </geometry>
-      <material name="${antenna_color}" />
-    </visual>
-    <collision>
-      <origin xyz="0 0 ${antenna_length/2}" rpy="0 0 0" />
-      <geometry>
-        <cylinder radius="${antenna_radius}" length="${antenna_length}" />
-      </geometry>
-    </collision>
-  </link>
-  <joint name="antenna_1_joint" type="fixed">
-    <parent link="chassis" />
-    <child link="antenna_1" />
-    <origin xyz="${antenna1_x} ${antenna1_y} ${antenna1_z}" rpy="0 0 0" />
-  </joint>
-  <!-- Вторая антенна (левая) -->
-  <link name="antenna_2">
-    <inertial>
-      <origin xyz="0 0 ${antenna_length/2}" rpy="0 0 0" />
-      <mass value="${antenna_mass}" />
-      <inertia
-        ixx="${(1/12) * antenna_mass * (3*antenna_radius*antenna_radius + antenna_length*antenna_length)}"
-        ixy="0.0" ixz="0.0"
-        iyy="${(1/12) * antenna_mass * (3*antenna_radius*antenna_radius + antenna_length*antenna_length)}"
-        iyz="0.0"
-        izz="${(1/2) * antenna_mass * antenna_radius*antenna_radius}" />
-    </inertial>
-    <visual>
-      <origin xyz="0 0 ${antenna_length/2}" rpy="0 0 0" />
-      <geometry>
-        <cylinder radius="${antenna_radius}" length="${antenna_length}" />
-      </geometry>
-      <material name="${antenna_color}" />
-    </visual>
-    <collision>
-      <origin xyz="0 0 ${antenna_length/2}" rpy="0 0 0" />
-      <geometry>
-        <cylinder radius="${antenna_radius}" length="${antenna_length}" />
-      </geometry>
-    </collision>
-  </link>
-  <joint name="antenna_2_joint" type="fixed">
-    <parent link="chassis" />
-    <child link="antenna_2" />
-    <origin xyz="${antenna2_x} ${antenna2_y} ${antenna2_z}" rpy="0 0 0" />
-  </joint>
-  <!-- Gazebo материалы для антенн -->
-  <gazebo reference="antenna_1">
-    <material>Gazebo/Black</material>
-  </gazebo>
-  <gazebo reference="antenna_2">
-    <material>Gazebo/Black</material>
-  </gazebo>
 </robot>
